File: greenecu48.kicad_pcb (KiCad board)
At the start: 4 copper layers, 128 x 110.6 mm, 2 parts, among them M1 Module-mega-mcu144-0.7, U1 molex_48pin_MRE

Commit message: wew
Parts:
- added C1: 10n, hellen-one-common:C0603, F.Cu at (205.2, 65.0)
- added C2: 100n, hellen-one-common:C0603, F.Cu at (194.5, 64.8)
- added C3: 10n, hellen-one-common:C0603, F.Cu at (197.5, 64.5)
- added C4: 100n, hellen-one-common:C0603, F.Cu at (195.6, 74.4)
- added C5: 1u, hellen-one-common:C0603, F.Cu at (195.6, 72.3)
- added D1: NUP2105L, Package_TO_SOT_SMD:SOT-23, F.Cu at (194.5, 68.2)
- added D10: 1N4148WS, hellen-one-common:SOD-323, F.Cu at (146.4, 78.8)
- added D11: LED-GREEN-0805, hellen-one-common:LED-0805, F.Cu at (146.9, 74.4)
- added D12: LED-GREEN-0805, hellen-one-common:LED-0805, F.Cu at (151.6, 78.8)
- added D13: LED-GREEN-0805, hellen-one-common:LED-0805, F.Cu at (189.5, 94.4)
- added D14: LED-GREEN-0805, hellen-one-common:LED-0805, F.Cu at (190.7, 97.9)
- added D2: B5819W, hellen-one-common:SOD-123, F.Cu at (171.3, 47.0)
- added D3: B5819W, hellen-one-common:SOD-123, F.Cu at (134.4, 68.0)
- added D4: B5819W, hellen-one-common:SOD-123, F.Cu at (133.3, 51.7)
- added D5: B5819W, hellen-one-common:SOD-123, F.Cu at (133.7, 57.8)
- added D9: 1N4148WS, hellen-one-common:SOD-323, F.Cu at (146.3, 76.7)
- added F10: Fuse-Pad-Pad, hellen-one-common:PAD-1206-PAD, F.Cu at (137.4, 50.6)
- added J4: USB_B_Mini, hellen-one-common:USB-MINI-B-VERTICAL, F.Cu at (125.4, 124.1)
- added L1: 470R@100MHz, Inductor_SMD:L_0603_1608Metric, F.Cu at (199.9, 64.5)
- added L2: 470R@100MHz, Inductor_SMD:L_0603_1608Metric, F.Cu at (202.9, 64.8)
- added M1: Module-power_12and5V-0.1, power-12-5v-0.1:power_12and5V, F.Cu at (141.4, 68.7)
- added M2: Module-vr-discrete-0.4, vr-discrete-0.4:vr-discrete, F.Cu at (177.9, 46.3)
- added M3: Module-knock-0.2, knock-0.2:knock, F.Cu at (173.2, 46.6)
- added M4: Module-ign8-0.2, ign8-0.2:ign8, F.Cu at (117.4, 110.3)
- added M5: Module-wbo-0.5, wbo-0.5:wbo, F.Cu at (204.2, 61.4)
- added M6: Module-can-0.1, can-01:can, F.Cu at (199.3, 95.7)
- added M7: Module-ign8-0.2, ign8-0.2:ign8, F.Cu at (134.3, 83.0)
- added Q11: ISL9V3040D3ST, Package_TO_SOT_SMD:TO-252-2, F.Cu at (125.6, 68.3)
- added Q12: ISL9V3040D3ST, Package_TO_SOT_SMD:TO-252-2, F.Cu at (192.6, 30.0)
- added Q14: ISL9V3040D3ST, Package_TO_SOT_SMD:TO-252-2, F.Cu at (124.9, 59.4)
- added Q9: ISL9V3040D3ST, Package_TO_SOT_SMD:TO-252-2, F.Cu at (124.9, 51.2)
- added Q901: ISL9V3040D3ST, Package_TO_SOT_SMD:TO-252-2, F.Cu at (89.2, 97.5)
- added Q902: ISL9V3040D3ST, Package_TO_SOT_SMD:TO-252-2, F.Cu at (89.2, 51.6)
- added Q903: ISL9V3040D3ST, Package_TO_SOT_SMD:TO-252-2, F.Cu at (99.9, 51.7)
- added Q904: ISL9V3040D3ST, Package_TO_SOT_SMD:TO-252-2, F.Cu at (89.4, 82.4)
- added Q905: ISL9V3040D3ST, Package_TO_SOT_SMD:TO-252-2, F.Cu at (110.4, 82.4)
- added Q906: ISL9V3040D3ST, Package_TO_SOT_SMD:TO-252-2, F.Cu at (89.0, 66.6)
- added Q911: ISL9V3040D3ST, Package_TO_SOT_SMD:TO-252-2, F.Cu at (99.7, 66.7)
- added Q912: ISL9V3040D3ST, Package_TO_SOT_SMD:TO-252-2, F.Cu at (99.8, 97.6)
- added Q913: ISL9V3040D3ST, Package_TO_SOT_SMD:TO-252-2, F.Cu at (110.3, 51.6)
- added Q914: ISL9V3040D3ST, Package_TO_SOT_SMD:TO-252-2, F.Cu at (110.2, 97.5)
- added Q915: ISL9V3040D3ST, Package_TO_SOT_SMD:TO-252-2, F.Cu at (110.0, 66.6)
- added Q916: ISL9V3040D3ST, Package_TO_SOT_SMD:TO-252-2, F.Cu at (120.9, 97.5)
- added R11: 22, hellen-one-common:R0603, F.Cu at (119.7, 59.4)
- added R12: 22, hellen-one-common:R0603, F.Cu at (119.6, 51.2)
- added R13: 5.1k, hellen-one-common:R0603, F.Cu at (148.3, 72.3)
- added R14: 5.1k, hellen-one-common:R0603, F.Cu at (151.7, 81.0)
- added R15: 1.6k, hellen-one-common:R0603, F.Cu at (195.0, 96.0)
- added R16: 750, hellen-one-common:R0603, F.Cu at (195.0, 98.2)
- added R17: 0, hellen-one-common:R0603, F.Cu at (118.7, 123.8)
- added R19: 22, hellen-one-common:R0603, F.Cu at (120.5, 68.3)
- added R401: 10k, hellen-one-common:R0603, B.Cu at (120.1, 120.4)
- added R402: 10k, hellen-one-common:R0603, B.Cu at (118.6, 120.4)
- added R403: 10k, hellen-one-common:R0603, B.Cu at (122.5, 120.4)
- added R404: 10k, hellen-one-common:R0603, B.Cu at (124.3, 120.4)
- added R405: 10k, hellen-one-common:R0603, B.Cu at (125.7, 120.4)
- added R406: 10k, hellen-one-common:R0603, B.Cu at (127.0, 120.2)
- added R9: 22, hellen-one-common:R0603, F.Cu at (186.9, 30.0)
- added R901: 22, hellen-one-common:R0603, B.Cu at (89.2, 102.5)
- added R902: 22, hellen-one-common:R0603, B.Cu at (89.3, 56.5)
- added R903: 22, hellen-one-common:R0603, B.Cu at (100.0, 56.6)
- added R904: 22, hellen-one-common:R0603, B.Cu at (89.4, 87.4)
- added R905: 22, hellen-one-common:R0603, B.Cu at (110.6, 87.1)
- added R906: 22, hellen-one-common:R0603, B.Cu at (89.1, 71.6)
- added R911: 22, hellen-one-common:R0603, B.Cu at (99.7, 71.7)
- added R912: 22, hellen-one-common:R0603, B.Cu at (99.9, 102.6)
- added R913: 22, hellen-one-common:R0603, B.Cu at (110.4, 55.9)
- added R914: 22, hellen-one-common:R0603, B.Cu at (110.2, 102.5)
- added R915: 22, hellen-one-common:R0603, B.Cu at (110.1, 71.2)
- added R916: 22, hellen-one-common:R0603, B.Cu at (121.0, 102.4)
- added U2: MAX31855KASA, Package_SO:SOIC-8_3.9x4.9mm_P1.27mm, F.Cu at (201.1, 70.3)
- M9: renamed from M1; footprint mega-144:mega-mcu144 -> mega-144-07:mega-mcu144
- moved M9 68.1 mm to (182.3, 83.7), turned to 180 degrees
Connections:
- M9 pad E1: unconnected-(M1-SPI2_SCK/CAN2_TX-PadE1) -> Net-(M6-CAN_TX)
- M9 pad E10: unconnected-(M1-OUT_IO10-PadE10) -> /VVT1_1
- M9 pad E12: unconnected-(M1-OUT_IO2-PadE12) -> /WASTEGATE
- M9 pad E13: unconnected-(M1-OUT_IO12-PadE13) -> /ETB_EN
- M9 pad E14: unconnected-(M1-OUT_PWM5-PadE14) -> /VVT2_B1
- M9 pad E15: unconnected-(M1-OUT_PWM4-PadE15) -> /VVT2_B2
- M9 pad E16: unconnected-(M1-OUT_PWM3-PadE16) -> /-ETB
- M9 pad E17: unconnected-(M1-OUT_PWM2-PadE17) -> /+ETB
- M9 pad E18: unconnected-(M1-OUT_INJ2-PadE18) -> /INJ2
- M9 pad E19: unconnected-(M1-OUT_INJ1-PadE19) -> /INJ1
- M9 pad E21: unconnected-(M1-OUT_IO4-PadE21) -> /IDLE
- M9 pad E22: unconnected-(M1-OUT_IO8-PadE22) -> /CHECK_ENGINE
- M9 pad E23: unconnected-(M1-OUT_IO7-PadE23) -> /VVT1_2
- M9 pad E25: unconnected-(M1-OUT_PWM7-PadE25) -> /FUEL_CONSUM
- M9 pad E26: unconnected-(M1-OUT_PWM6-PadE26) -> /THRESHOLD_VR
- M9 pad E27: unconnected-(M1-OUT_PWM1-PadE27) -> /TACH
- M9 pad E28: unconnected-(M1-OUT_PWM8-PadE28) -> /OUT3
- M9 pad E29: unconnected-(M1-OUT_INJ3-PadE29) -> /INJ3
- M9 pad E30: unconnected-(M1-OUT_INJ4-PadE30) -> /INJ4
- M9 pad E31: unconnected-(M1-OUT_INJ5-PadE31) -> /INJ5
- M9 pad E32: unconnected-(M1-OUT_INJ6-PadE32) -> /INJ6
- M9 pad E4: unconnected-(M1-SPI2_CS/CAN2_RX-PadE4) -> Net-(M6-CAN_RX)
- M9 pad E6: unconnected-(M1-OUT_IO3-PadE6) -> /MAIN_RELAY
- M9 pad E7: unconnected-(M1-OUT_IO5-PadE7) -> /OUT1
- M9 pad E8: unconnected-(M1-OUT_IO1-PadE8) -> /FUEL_PUMP_RELAY
- M9 pad E9: unconnected-(M1-OUT_IO6-PadE9) -> /OUT2
- M9 pad G: unconnected-(M1-GND-PadG) -> GND
- M9 pad N10: unconnected-(M1-SPI3_CS-PadN10) -> /SPI3_CS
- M9 pad N11: unconnected-(M1-SPI3_SCK-PadN11) -> /SPI3_SCK
- M9 pad N12: unconnected-(M1-SPI3_MISO-PadN12) -> /SPI3_MISO
- M9 pad N13: unconnected-(M1-SPI3_MOSI-PadN13) -> /SPI3_MOSI
- M9 pad N17: unconnected-(M1-UART2_TX-PadN17) -> /TX2
- M9 pad N18: unconnected-(M1-UART2_RX-PadN18) -> /RX2
- M9 pad N2: unconnected-(M1-USBM-PadN2) -> /USBM
- M9 pad N24: unconnected-(M1-UART8_RX-PadN24) -> /RX1
- M9 pad N25: unconnected-(M1-UART8_TX-PadN25) -> /TX1
- M9 pad N26: unconnected-(M1-IN_VIGN-PadN26) -> /VIGN
- M9 pad N27: unconnected-(M1-VBAT-PadN27) -> /VBAT
- M9 pad N3: unconnected-(M1-USBP-PadN3) -> /USBP
- M9 pad N30: unconnected-(M1-V5A_SWITCHABLE-PadN30) -> +5VA
- M9 pad N31: unconnected-(M1-VCC-PadN31) -> +5V
- M9 pad N32: unconnected-(M1-V33-PadN32) -> +3V3
- M9 pad N4: unconnected-(M1-VBUS-PadN4) -> /VBUS
- M9 pad S1: unconnected-(M1-IN_D4-PadS1) -> /IN_D4
- M9 pad S10: unconnected-(M1-IN_AUX4-PadS10) -> /IN_CAM2
- M9 pad S11: unconnected-(M1-IN_AUX3-PadS11) -> /IN_A3
- M9 pad S12: unconnected-(M1-IN_AUX2-PadS12) -> /IN_PPS2
- M9 pad S13: unconnected-(M1-IN_AUX1-PadS13) -> /IN_TPS2
- M9 pad S14: unconnected-(M1-IN_RES2-PadS14) -> /IN_RES2
- M9 pad S15: unconnected-(M1-IN_O2S2-PadS15) -> /IN_A1
- M9 pad S16: unconnected-(M1-IN_O2S-PadS16) -> /IN_AFR
- M9 pad S17: unconnected-(M1-IN_RES1-PadS17) -> /IN_RES1
- M9 pad S18: unconnected-(M1-IN_RES3-PadS18) -> /IN_A4
- M9 pad S19: unconnected-(M1-IN_MAP3-PadS19) -> /IN_A2
- M9 pad S2: unconnected-(M1-IN_D3-PadS2) -> /IN_D3
- M9 pad S20: unconnected-(M1-IN_MAP2-PadS20) -> /IN_MAP2
- M9 pad S21: unconnected-(M1-IN_MAP1-PadS21) -> /IN_MAF
- M9 pad S22: unconnected-(M1-IN_CRANK-PadS22) -> /IN_CRANK
- M9 pad S23: unconnected-(M1-IN_KNOCK-PadS23) -> /IN_KNOCK1
- M9 pad S24: unconnected-(M1-IN_CAM-PadS24) -> /IN_CAM1
- M9 pad S25: unconnected-(M1-IN_VSS-PadS25) -> /IN_VSS
- M9 pad S26: unconnected-(M1-IN_IAT-PadS26) -> /IN_IAT
- M9 pad S28: unconnected-(M1-IN_CLT-PadS28) -> /IN_CLT
- M9 pad S3: unconnected-(M1-IN_D2-PadS3) -> /IN_D2
- M9 pad S30: unconnected-(M1-IN_TPS-PadS30) -> /IN_TPS1
- M9 pad S31: unconnected-(M1-IN_PPS-PadS31) -> /IN_PPS1
- M9 pad S4: unconnected-(M1-IN_D1-PadS4) -> /IN_D1
- M9 pad S5: unconnected-(M1-VREF2-PadS5) -> /VREF2
- M9 pad S9: unconnected-(M1-IN_SENS1-PadS9) -> /VR_ANALOG
- M9 pad W1: unconnected-(M1-GNDA-PadW1) -> /GNDA
- M9 pad W10: unconnected-(M1-IGN2-PadW10) -> /IGN2
- M9 pad W11: unconnected-(M1-IGN1-PadW11) -> /IGN1
- M9 pad W12: unconnected-(M1-CANH-PadW12) -> /CAN+
- M9 pad W13: unconnected-(M1-CANL-PadW13) -> /CAN-
- M9 pad W6: unconnected-(M1-IGN6-PadW6) -> /IGN6
- M9 pad W7: unconnected-(M1-IGN5-PadW7) -> /IGN5
- M9 pad W8: unconnected-(M1-IGN4-PadW8) -> /IGN4
- M9 pad W9: unconnected-(M1-IGN3-PadW9) -> /IGN3
- U1 pad 1: /12V_MREL -> /OUT_IGN1
- U1 pad 10: /Ign2 -> /OUT_INJ3
- U1 pad 11: /Ign3 -> /OUT_INJ5
- U1 pad 12: /Ign4 -> +12V
- U1 pad 13: /GP6 -> /OUT_INJ2
- U1 pad 14: /GP5 -> /OUT_INJ4
- U1 pad 15: /USB_D- -> /OUT_INJ6
- U1 pad 16: /USB_D+ -> +12V
- U1 pad 17: /GND -> /LSU_SENSOR_U
- U1 pad 18: /AT1 -> /LSU_PUMP_I
- U1 pad 19: /AV4 -> /IN_MAP2
- U1 pad 2: /GND -> /OUT_IGN3
- U1 pad 20: /AV5 -> /IN_CAM1
- U1 pad 21: /GND -> /LSU_CALIBR_RES
- U1 pad 22: /AT4 -> /LSU_HEAT-
- U1 pad 23: /AT2 -> /IN_IAT
- U1 pad 24: /AT3 -> /IN_CLT
- U1 pad 25: /CAM_SENSOR -> /LSU_SENSOR_U/PUMP_I
- U1 pad 26: /AV2 -> /IN_CRANK+
- U1 pad 27: /AV1 -> /IN_TPS1
- U1 pad 28: /AV10 -> /IN_PPS1
- U1 pad 29: /MAIN_RELAY -> /IN_CRANK-
- U1 pad 3: /LS2 -> /OUT_IGN5
- U1 pad 30: /AV7 -> +5VP
- U1 pad 31: /AV3 -> +5VP
- U1 pad 32: /AV6 -> /OUT_TACH
- U1 pad 33: /GP3 -> /IN_KNOCK1_RAW
- U1 pad 34: /GP2 -> /CAN_L
- U1 pad 35: /GP1 -> /USBM
- U1 pad 36: /AV8 -> /OUT_BUZER
- U1 pad 37: /INJECTOR-1 -> /GNDA
- U1 pad 38: /INJECTOR-2 -> /GNDA
- U1 pad 39: /5V2 -> /CAN_H
- U1 pad 4: /E-THROTTLE+ -> GND
- U1 pad 40: /AV9 -> /USBP
- U1 pad 41: /INJECTOR-3 -> /GNDA
- U1 pad 42: /INJECTOR-4 -> /GNDA
- U1 pad 43: /GP4 -> /EGT-
- U1 pad 44: /5V1 -> /OUT_WASTEGATE
- U1 pad 45: /CRNK+ -> /GNDA
- U1 pad 46: /CRNK- -> /GNDA
- U1 pad 47: /CANL -> /EGT+
- U1 pad 48: /CANH -> /OUT_FUEL_PUMP_RELAY
- U1 pad 5: /12V_KEY -> /OUT_IGN2
- U1 pad 6: /GND -> /OUT_IGN4
- U1 pad 7: /LS1 -> /OUT_IGN6
- U1 pad 8: /E-THROTTLE- -> GND
- U1 pad 9: /Ign1 -> /OUT_INJ1
Routing:
- net Net-(M7-OUT_IGN4): track 0.00 -> 227.5 mm, vias 0 -> 3
- net /IGN3: track 0.00 -> 202.3 mm, vias 0 -> 3
- net /OUT_IGN6: track 0.00 -> 200.3 mm, vias 0 -> 10
- net /IGN5: track 0.00 -> 194.8 mm, vias 0 -> 3
- net /OUT_INJ5: track 0.00 -> 193.2 mm, vias 0 -> 10
- net +5VA: track 0.00 -> 191.8 mm, vias 0 -> 4
- net /OUT_IGN4: track 0.00 -> 178.6 mm, vias 0 -> 10
- net /IGN1: track 0.00 -> 175.1 mm, vias 0 -> 3
- net /OUT_INJ4: track 0.00 -> 172.1 mm, vias 0 -> 10
- net /IGN6: track 0.00 -> 171.8 mm, vias 0 -> 3
- net /OUT_INJ1: track 0.00 -> 169.6 mm, vias 0 -> 10
- net +3V3: track 0.00 -> 164.9 mm, vias 0 -> 5
- net /OUT_INJ6: track 0.00 -> 162.0 mm, vias 0 -> 10
- net /OUT_IGN2: track 0.00 -> 159.8 mm, vias 0 -> 10
- net /IGN4: track 0.00 -> 157.8 mm, vias 0 -> 3
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- added copper zone on B.Cu, net /OUT_IGN1
- added copper zone on B.Cu, net /OUT_IGN2
- added copper zone on B.Cu, net /OUT_IGN3
- added copper zone on B.Cu, net /OUT_IGN4
- added copper zone on B.Cu, net /OUT_IGN5
- added copper zone on B.Cu, net /OUT_IGN6
- added copper zone on B.Cu, net /OUT_INJ1
- added copper zone on B.Cu, net /OUT_INJ2
- added copper zone on B.Cu, net /OUT_INJ3
- added copper zone on B.Cu, net /OUT_INJ4
- added copper zone on B.Cu, net /OUT_INJ5
- added copper zone on B.Cu, net /OUT_INJ6
- added copper zone on B.Cu, net GND
- added copper zone on F.Cu, net GND
- added copper zone on In1.Cu, net GND
- added copper zone on In2.Cu, net GND
