File: greenecu48.kicad_pcb (KiCad board)
At the start: 4 copper layers, 128 x 110.6 mm, 73 parts, among them J4 USB_B_Mini, M1 Module-power_12and5V-0.1, M2 Module-vr-discrete-0.4, M3 Module-knock-0.2, M4 Module-ign8-0.2, M5 Module-wbo-0.5, M6 Module-can-0.1, M7 Module-ign8-0.2, M9 Module-mega-mcu144-0.7, Q11 ISL9V3040D3ST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

Commit message: gshw
Parts:
- added G***: LOGO, GDI-6ch:lokone, F.Cu at (160.3, 128.5)
- added G***: LOGO, GDI-6ch:lokone, B.Cu at (160.3, 128.5)
Other:
- outline, holes or cut-outs redrawn

Commit message: qwq
Parts:
- removed G*** (x2): LOGO, GDI-6ch:lokone

Commit message: wew
Parts:
- added G***: LOGO, GDI-6ch:lokone, F.Cu at (158.8, 129.5)
- added G***: LOGO, GDI-6ch:lokone, B.Cu at (158.8, 129.5)
