File: greenecu48.kicad_sch (KiCad schematic)
At the start: 2 parts, among them M1 Module-mega-mcu144-0.7, U1 molex_48pin_MRE

Commit message: wew
Parts:
- removed M1: Module-mega-mcu144-0.7, mega-144:mega-mcu144, symbol mega-mcu144:Module-mega-mcu144-0.7
- added D10, D9: 1N4148WS, hellen-one-common:SOD-323, symbol hellen-one-common:1N4148WS
- added D11, D12, D13, D14: LED-GREEN-0805, hellen-one-common:LED-0805, symbol hellen-one-common:LED
- added D2, D3, D4, D5: B5819W, hellen-one-common:SOD-123, symbol hellen-one-common:1N4148WS
- added F10: Fuse-Pad-Pad, hellen-one-common:PAD-1206-PAD, symbol hellen-one-common:Fuse-Pad-Pad
- added J4: USB_B_Mini, hellen-one-common:USB-MINI-B-VERTICAL, symbol hellen-one-common:USB_B_Mini
- added M1: Module-power_12and5V-0.1, power-12-5v-0.1:power_12and5V, symbol power_12and5V-0.1:Module-power_12and5V-0.1
- added M2: Module-vr-discrete-0.4, vr-discrete-0.4:vr-discrete, symbol vr-discrete-0.4:Module-vr-discrete-0.4
- added M3: Module-knock-0.2, knock-0.2:knock, symbol hellen-one-knock-0.2:Module-knock-0.2
- added M5: Module-wbo-0.5, wbo-0.5:wbo, symbol hellen-one-wbo-0.5:Module-wbo-0.5
- added M6: Module-can-0.1, can-01:can, symbol can:Module-can-0.1
- added M9: Module-mega-mcu144-0.7, mega-144-07:mega-mcu144, symbol mega-mcu144:Module-mega-mcu144-0.7
- added R13, R14: 5.1k, hellen-one-common:R0603, symbol hellen-one-common:Res
- added R15: 1.6k, hellen-one-common:R0603, symbol hellen-one-common:Res
- added R16: 750, hellen-one-common:R0603, symbol hellen-one-common:Res
- added R17: 0, hellen-one-common:R0603, symbol hellen-one-common:Res
Connections:
- net AV7 is gone; now on net +5VP: U1.30
- net CRNK- is gone; now on net GNDA: U1.46
- net E-THROTTLE+ is gone; now on net GND: U1.4
- net E-THROTTLE- is gone; now on net GND: U1.8
- net INJECTOR-1 is gone; now on net GNDA: U1.37
- net INJECTOR-2 is gone; now on net GNDA: U1.38
- net INJECTOR-3 is gone; now on net GNDA: U1.41
- net INJECTOR-4 is gone; now on net GNDA: U1.42
- net USB_D+ is gone; now on net +12V: U1.16
- net GND: now also M1.S1 (GND), M2.G (GND), M3.E2 (GND), M5.E6 (LSU_H-), M5.G (GND), M6.E1 (GND), M9.G (GND), R13.2, R14.2, R15.2, R16.2, R17.2; no longer U1.17, U1.2, U1.21, U1.6
- net MAIN_RELAY: now also M9.E6 (OUT_IO3); no longer U1.29
- net 12V_KEY renamed OUT_IGN2
- net 12V_MREL renamed OUT_IGN1
- net 5V1 renamed OUT_WASTEGATE
- net OUT_WASTEGATE: now also D3.2 (A)
- net 5V2 renamed CAN_H
- net CAN_H: now also M6.S2 (CANH)
- net AT1 renamed LSU_PUMP_I
- net LSU_PUMP_I: now also M5.E3 (LSU_Ip)
- net AT2 renamed IN_IAT
- net IN_IAT: now also M9.S26 (IN_IAT)
- net AT3 renamed IN_CLT
- net IN_CLT: now also M9.S28 (IN_CLT)
- net AT4 renamed LSU_HEAT-
- net LSU_HEAT-: now also M5.E5 (LSU_H+)
- net AV1 renamed IN_TPS1
- net IN_TPS1: now also M9.S30 (IN_TPS)
- net AV10 renamed IN_PPS1
- net IN_PPS1: now also M9.S31 (IN_PPS)
- net AV2 renamed IN_CRANK+
- net IN_CRANK+: now also M2.W2 (VR+)
- net AV3 renamed +5VP
- net +5VP: now also M1.V4 (5VP)
- net AV4 renamed IN_MAP2
- net IN_MAP2: now also M9.S20 (IN_MAP2)
- net AV5 renamed IN_CAM1
- net IN_CAM1: now also M9.S24 (IN_CAM)
- net AV6 renamed OUT_TACH
- net OUT_TACH: now also D4.2 (A)
- net AV8 renamed OUT_BUZER
- net OUT_BUZER: now also D5.2 (A)
- net AV9 renamed USBP
- net USBP: now also J4.3 (D+), M9.N3 (USBP)
- net CAM_SENSOR renamed LSU_SENSOR_U/PUMP_I
- net LSU_SENSOR_U/PUMP_I: now also M5.E2 (LSU_Vm)
- net CANH renamed OUT_FUEL_PUMP_RELAY
- net OUT_FUEL_PUMP_RELAY: now also D2.2 (A)
- net CANL renamed EGT+
- net CRNK+ renamed GNDA
- net GNDA: now also M9.W1 (GNDA)
- net GP1 renamed USBM
- net USBM: now also J4.2 (D-), M9.N2 (USBM)
- net GP2 renamed CAN_L
- net CAN_L: now also M6.S1 (CANL)
- net GP3 renamed IN_KNOCK1_RAW
- net IN_KNOCK1_RAW: now also M3.W1 (IN_KNOCK)
- net GP4 renamed EGT-
- net GP5 renamed OUT_INJ4
- net GP6 renamed OUT_INJ2
- net Ign1 renamed OUT_INJ1
- net Ign2 renamed OUT_INJ3
- net Ign3 renamed OUT_INJ5
- net Ign4 renamed +12V
- net +12V: now also D10.1 (K), D11.1 (A), D12.1 (A), D2.1 (K), D3.1 (K), D4.1 (K), D5.1 (K), D9.1 (K), F10.1, M1.E2 (V12)
- net LS1 renamed OUT_IGN6
- net LS2 renamed OUT_IGN5
- net USB_D- renamed OUT_INJ6
- new net: D11.2 (K), D9.2 (A), R13.1
- new net: D13.2 (K), R15.1
- new net: D14.2 (K), R16.1
- new net: J4.5 (GND), J4.6 (Shield), R17.1
- new net: D10.2 (A), D12.2 (K), R14.1
- new net: M6.V5 (CAN_TX), M9.E1 (SPI2_SCK/CAN2_TX)
- new net: M6.V6 (CAN_RX), M9.E4 (SPI2_CS/CAN2_RX)
- new net: M5.J2 (SEL2), M5.J_VCC2 (PULL_UP2)
- new net +12V_PROT: M1.E5 (EN_5VP)
- new net +12V_RAW: F10.2, M1.V1 (V12_PERM), M1.V2 (IN_VIGN), M1.V3 (V12_RAW)
- new net +3V3: D14.1 (A), M6.V2 (CAN_VIO), M9.N32 (V33)
- new net +5V: D13.1 (A), M1.E4 (V5), M2.E4 (V5_IN), M5.W1 (V5_IN), M9.N31 (VCC)
- new net +5VA: M3.E1 (V5A), M6.V1 (V5), M9.N30 (V5A_SWITCHABLE)
- new net +ETB: M9.E17 (OUT_PWM2)
- new net -ETB: M9.E16 (OUT_PWM3)
- new net CAN+: M5.W4 (CANH), M9.W12 (CANH)
- new net CAN-: M5.W3 (CANL), M9.W13 (CANL)
- new net CHECK_ENGINE: M9.E22 (OUT_IO8)
- new net ETB_EN: M9.E13 (OUT_IO12)
- new net FUEL_CONSUM: M9.E25 (OUT_PWM7)
- new net FUEL_PUMP_RELAY: M9.E8 (OUT_IO1)
- new net IDLE: M9.E21 (OUT_IO4)
- new net IGN1: M9.W11 (IGN1)
- new net IGN2: M9.W10 (IGN2)
- new net IGN3: M9.W9 (IGN3)
- new net IGN4: M9.W8 (IGN4)
- new net IGN5: M9.W7 (IGN5)
- new net IGN6: M9.W6 (IGN6)
- new net INJ1: M9.E19 (OUT_INJ1)
- new net INJ2: M9.E18 (OUT_INJ2)
- new net INJ3: M9.E29 (OUT_INJ3)
- new net INJ4: M9.E30 (OUT_INJ4)
- new net INJ5: M9.E31 (OUT_INJ5)
- new net INJ6: M9.E32 (OUT_INJ6)
- new net IN_A1: M9.S15 (IN_O2S2)
- new net IN_A2: M9.S19 (IN_MAP3)
- new net IN_A3: M9.S11 (IN_AUX3)
- new net IN_A4: M9.S18 (IN_RES3)
- new net IN_AFR: M9.S16 (IN_O2S)
- new net IN_CAM2: M9.S10 (IN_AUX4)
- new net IN_CRANK: M2.E3 (OUT), M9.S22 (IN_CRANK)
- new net IN_CRANK-: M2.W1 (VR-), U1.29
- new net IN_D1: M9.S4 (IN_D1)
- new net IN_D2: M9.S3 (IN_D2)
- new net IN_D3: M9.S2 (IN_D3)
- new net IN_D4: M9.S1 (IN_D4)
- new net IN_KNOCK1: M3.E3 (OUT_KNOCK), M9.S23 (IN_KNOCK)
- new net IN_MAF: M9.S21 (IN_MAP1)
- new net IN_PPS2: M9.S12 (IN_AUX2)
- new net IN_RES1: M9.S17 (IN_RES1)
- new net IN_RES2: M9.S14 (IN_RES2)
- new net IN_TPS2: M9.S13 (IN_AUX1)
- new net IN_VSS: M9.S25 (IN_VSS)
- new net LSU_CALIBR_RES: M5.E4 (LSU_Rtrim), U1.21
- new net LSU_SENSOR_U: M5.E1 (LSU_Un), U1.17
- new net OUT1: M9.E7 (OUT_IO5)
- new net OUT2: M9.E9 (OUT_IO6)
- new net OUT3: M9.E28 (OUT_PWM8)
- new net OUT_IGN3: U1.2
- new net OUT_IGN4: U1.6
- new net RX1: M9.N24 (UART8_RX)
- new net RX2: M9.N18 (UART2_RX)
- new net SPI3_CS: M9.N10 (SPI3_CS)
- new net SPI3_MISO: M9.N12 (SPI3_MISO)
- new net SPI3_MOSI: M9.N13 (SPI3_MOSI)
- new net SPI3_SCK: M9.N11 (SPI3_SCK)
- new net TACH: M9.E27 (OUT_PWM1)
- new net THRESHOLD_VR: M2.E1 (Thresh_IN), M9.E26 (OUT_PWM6)
- new net TX1: M9.N25 (UART8_TX)
- new net TX2: M9.N17 (UART2_TX)
- new net VBAT: M9.N27 (VBAT)
- new net VBUS: J4.1 (VBUS), M9.N4 (VBUS)
- new net VIGN: M1.E3 (VIGN), M9.N26 (IN_VIGN)
- new net VREF2: M3.W2 (VREF), M9.S5 (VREF2)
- new net VR_ANALOG: M2.E2 (OUT_A), M9.S9 (IN_SENS1)
- new net VVT1_1: M9.E10 (OUT_IO10)
- new net VVT1_2: M9.E23 (OUT_IO7)
- new net VVT2_B1: M9.E14 (OUT_PWM5)
- new net VVT2_B2: M9.E15 (OUT_PWM4)
- new net WASTEGATE: M9.E12 (OUT_IO2)
- no-connect marks 0 -> 45
Other:
- added sheet EGT (egt.kicad_sch)
- added sheet Ignition (IGN6.kicad_sch)
- added sheet Injector (INJ6.kicad_sch)
- added sheet LOW_SIDE (LOW_SIDE.kicad_sch)
- note added: "#1"
- note added: "Flyback diodes"
- note added: "LEDs"
- note added: "Power"
- moved on the sheet: U1A
