File: greenecu48.kicad_sch (KiCad schematic)
At the start: 24 parts, among them J4 USB_B_Mini, M1 Module-power_12and5V-0.1, M2 Module-vr-discrete-0.4, M3 Module-knock-0.2, M5 Module-wbo-0.5, M6 Module-can-0.1, M9 Module-mega-mcu144-0.7, U1 molex_48pin_MRE

Commit message: Actualizacion diseño greenecu48
Parts:
- added M8: Module-vr-max9924-0.1, vr-max9924-0.1:vr-max9924, symbol vr-max9924:Module-vr-max9924-0.1
Connections:
- net +12V_PROT: no longer M1.E5 (EN_5VP)
- net +5V: now also M1.E5 (EN_5VP), M8.E4 (V5_IN); no longer M2.E4 (V5_IN)
- net GND: now also M8.G (GND); no longer M2.G (GND)
- net IN_CRANK: now also M8.E3 (OUT); no longer M2.E3 (OUT)
- net IN_CRANK+: now also M8.W2 (VR+); no longer M2.W2 (VR+)
- net IN_CRANK-: now also M8.W1 (VR-); no longer M2.W1 (VR-)
- net THRESHOLD_VR: now also M8.E1 (NC); no longer M2.E1 (Thresh_IN)
- net VR_ANALOG: now also M8.E2 (NC); no longer M2.E2 (OUT_A)
Other:
- moved on the sheet: M2

Commit message: rede
Parts:
- U1: LCSC (none) -> C164171
Changed lines of the file:
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@@
 			)
 		)
-		(property "LCSC" ""
+		(property "LCSC" "C164171"
 			(at 565.15 67.945 0)
 			(effects
